File: PowerBoard/Boost/PowerBoard-Boost-v2.sch (KiCad schematic (older format))
At the start: 25 parts, among them J302 2X10-2MMSMD, M301 MOSFET_NSI4778DY, U301 LM3488

Commit message: Cleanup to assemble the power board V2.
Parts:
- CBP301, CCOMP302, COUT301, COUT302, COUT303: symbol PowerBoard-Boost-v2-eagle-import:C-USC1206 -> PowerBoth-rescue:C-USC1206-PowerBoard-Boost-v2-eagle-import
- CCOMP301, CFILT301, CSEP301, CSEP302: symbol PowerBoard-Boost-v2-eagle-import:C-USC0805 -> PowerBoth-rescue:C-USC0805-PowerBoard-Boost-v2-eagle-import
- CIN301, CIN302: symbol PowerBoard-Boost-v2-eagle-import:CPOL-US153CLV-0505 -> PowerBoth-rescue:CPOL-US153CLV-0505-PowerBoard-Boost-v2-eagle-import
- D301: symbol PowerBoard-Boost-v2-eagle-import:SL44-E3_57TDIODE_DO214AB-M -> PowerBoth-rescue:SL44-E3_57TDIODE_DO214AB-M-PowerBoard-Boost-v2-eagle-import
- J302: symbol PowerBoard-Boost-v2-eagle-import:2X10-2MMSMD -> PowerBoth-rescue:2X10-2MMSMD-PowerBoard-Boost-v2-eagle-import
- L301: symbol PowerBoard-Boost-v2-eagle-import:INDUCTOR_DUAL -> PowerBoth-rescue:INDUCTOR_DUAL-PowerBoard-Boost-v2-eagle-import
- M301: symbol PowerBoard-Boost-v2-eagle-import:MOSFET_NSI4778DY -> PowerBoth-rescue:MOSFET_NSI4778DY-PowerBoard-Boost-v2-eagle-import
- RBP301, RCOMP301, RFADJ301: symbol PowerBoard-Boost-v2-eagle-import:R-US_R0805 -> PowerBoth-rescue:R-US_R0805-PowerBoard-Boost-v2-eagle-import
- RFB301, RFB302, RFILT301, RSENSE301: symbol PowerBoard-Boost-v2-eagle-import:R-US_R1206 -> PowerBoth-rescue:R-US_R1206-PowerBoard-Boost-v2-eagle-import
- TP301, TP302: symbol PowerBoard-Boost-v2-eagle-import:TEST_POINTROUND-1MM -> PowerBoth-rescue:TEST_POINTROUND-1MM-PowerBoard-Boost-v2-eagle-import
- U301: symbol PowerBoard-Boost-v2-eagle-import:LM3488QMM_NOPBDGK8-M -> PowerBoth-rescue:LM3488QMM_NOPBDGK8-M-PowerBoard-Boost-v2-eagle-import
Changed lines of the file:
@@
 Connection ~ 10000 1250
 $Comp
-L PowerBoard-Boost-v2-eagle-import:LM3488QMM_NOPBDGK8-M U?
+L PowerBoth-rescue:LM3488QMM_NOPBDGK8-M-PowerBoard-Boost-v2-eagle-import U?
 U 1 1 5ECBF6F0
 P 3500 1500
@@
 $EndComp
 $Comp
-L PowerBoard-Boost-v2-eagle-import:INDUCTOR_DUAL L?
+L PowerBoth-rescue:INDUCTOR_DUAL-PowerBoard-Boost-v2-eagle-import L?
 U 1 1 5ECBF6F6
 P 7750 3150
@@
 $EndComp
 $Comp
-L PowerBoard-Boost-v2-eagle-import:C-USC1206 COUT?
+L PowerBoth-rescue:C-USC1206-PowerBoard-Boost-v2-eagle-import COUT?
 U 1 1 5ECBF6FC
 P 10550 4850
@@
 $EndComp
 $Comp
-L PowerBoard-Boost-v2-eagle-import:C-USC1206 COUT?
+L PowerBoth-rescue:C-USC1206-PowerBoard-Boost-v2-eagle-import COUT?
 U 1 1 5ECBF702
 P 9550 4850
@@
 $EndComp
 $Comp
-L PowerBoard-Boost-v2-eagle-import:C-USC1206 COUT?
+L PowerBoth-rescue:C-USC1206-PowerBoard-Boost-v2-eagle-import COUT?
 U 1 1 5ECBF708
 P 10050 4850
@@
 $EndComp
 $Comp
-L PowerBoard-Boost-v2-eagle-import:C-USC0805 CCOMP?
+L PowerBoth-rescue:C-USC0805-PowerBoard-Boost-v2-eagle-import CCOMP?
 U 1 1 5ECBF70E
 P 3150 6400
@@
 $EndComp
 $Comp
-L PowerBoard-Boost-v2-eagle-import:R-US_R1206 RFB?
+L PowerBoth-rescue:R-US_R1206-PowerBoard-Boost-v2-eagle-import RFB?
 U 1 1 5ECBF714
 P 8850 4450
@@
 $EndComp
 $Comp
-L PowerBoard-Boost-v2-eagle-import:C-USC0805 CFILT?
+L PowerBoth-rescue:C-USC0805-PowerBoard-Boost-v2-eagle-import CFILT?
 U 1 1 5ECBF71A
 P 5450 5550
@@
 $EndComp
 $Comp
-L PowerBoard-Boost-v2-eagle-import:R-US_R1206 RSENSE?
+L PowerBoth-rescue:R-US_R1206-PowerBoard-Boost-v2-eagle-import RSENSE?
 U 1 1 5ECBF720
 P 6350 5550
@@
 $EndComp
 $Comp
-L PowerBoard-Boost-v2-eagle-import:C-USC1206 CCOMP?
+L PowerBoth-rescue:C-USC1206-PowerBoard-Boost-v2-eagle-import CCOMP?
 U 1 1 5ECBF726
 P 3650 6400
@@
 $EndComp
 $Comp
-L PowerBoard-Boost-v2-eagle-import:C-USC0805 CSEP?
+L PowerBoth-rescue:C-USC0805-PowerBoard-Boost-v2-eagle-import CSEP?
 U 1 1 5ECBF72C
 P 7850 3750
@@
 $EndComp
 $Comp
-L PowerBoard-Boost-v2-eagle-import:C-USC0805 CSEP?
+L PowerBoth-rescue:C-USC0805-PowerBoard-Boost-v2-eagle-import CSEP?
 U 1 1 5ECBF732
 P 7850 4250
@@
 $EndComp
 $Comp
-L PowerBoard-Boost-v2-eagle-import:R-US_R1206 RFB?
+L PowerBoth-rescue:R-US_R1206-PowerBoard-Boost-v2-eagle-import RFB?
 U 1 1 5ECBF738
 P 8850 5350
@@
 $EndComp
 $Comp
-L PowerBoard-Boost-v2-eagle-import:C-USC1206 CBP?
+L PowerBoth-rescue:C-USC1206-PowerBoard-Boost-v2-eagle-import CBP?
 U 1 1 5ECBF73E
 P 2550 6100
@@
 $EndComp
 $Comp
-L PowerBoard-Boost-v2-eagle-import:R-US_R1206 RFILT?
+L PowerBoth-rescue:R-US_R1206-PowerBoard-Boost-v2-eagle-import RFILT?
 U 1 1 5ECBF744
 P 5750 4950
@@
 $EndComp
 $Comp
-L PowerBoard-Boost-v2-eagle-import:R-US_R0805 RFADJ?
+L PowerBoth-rescue:R-US_R0805-PowerBoard-Boost-v2-eagle-import RFADJ?
 U 1 1 5ECBF74A
 P 4450 5900
@@
 $EndComp
 $Comp
-L PowerBoard-Boost-v2-eagle-import:R-US_R0805 RBP?
+L PowerBoth-rescue:R-US_R0805-PowerBoard-Boost-v2-eagle-import RBP?
 U 1 1 5ECBF750
 P 2550 5300
@@
 $EndComp
 $Comp
-L PowerBoard-Boost-v2-eagle-import:R-US_R0805 RCOMP?
+L PowerBoth-rescue:R-US_R0805-PowerBoard-Boost-v2-eagle-import RCOMP?
 U 1 1 5ECBF756
 P 3650 5700
@@
 $EndComp
 $Comp
-L PowerBoard-Boost-v2-eagle-import:MOSFET_NSI4778DY M?
+L PowerBoth-rescue:MOSFET_NSI4778DY-PowerBoard-Boost-v2-eagle-import M?
 U 1 1 5ECBF75C
 P 6350 4450
@@
 $EndComp
 $Comp
-L PowerBoard-Boost-v2-eagle-import:SL44-E3_57TDIODE_DO214AB-M D?
+L PowerBoth-rescue:SL44-E3_57TDIODE_DO214AB-M-PowerBoard-Boost-v2-eagle-import D?
 U 1 1 5ECBF762
 P 8450 4050
@@
 $EndComp
 $Comp
-L PowerBoard-Boost-v2-eagle-import:CPOL-US153CLV-0505 CIN?
+L PowerBoth-rescue:CPOL-US153CLV-0505-PowerBoard-Boost-v2-eagle-import CIN?
 U 1 1 5ECBF768
 P 1650 5300
@@
 $EndComp
 $Comp
-L PowerBoard-Boost-v2-eagle-import:CPOL-US153CLV-0505 CIN?
+L PowerBoth-rescue:CPOL-US153CLV-0505-PowerBoard-Boost-v2-eagle-import CIN?
 U 1 1 5ECBF76E
 P 2050 5300
@@
 $EndComp
 $Comp
-L PowerBoard-Boost-v2-eagle-import:GND #GND?
+L PowerBoth-rescue:GND-PowerBoard-Boost-v2-eagle-import #GND?
 U 1 1 5ECBF774
 P 1850 7300
@@
 $EndComp
 $Comp
-L PowerBoard-Boost-v2-eagle-import:GND #GND?
+L PowerBoth-rescue:GND-PowerBoard-Boost-v2-eagle-import #GND?
 U 1 1 5ECBF77A
 P 5000 3800
@@
 $EndComp
 $Comp
-L PowerBoard-Boost-v2-eagle-import:GND #GND?
+L PowerBoth-rescue:GND-PowerBoard-Boost-v2-eagle-import #GND?
 U 1 1 5ECBF780
 P 5850 6150
@@
 $EndComp
 $Comp
-L PowerBoard-Boost-v2-eagle-import:GND #GND?
+L PowerBoth-rescue:GND-PowerBoard-Boost-v2-eagle-import #GND?
 U 1 1 5ECBF786
 P 8250 5950
@@
 $EndComp
 $Comp
-L PowerBoard-Boost-v2-eagle-import:5V #SUPPLY?
+L PowerBoth-rescue:5V-PowerBoard-Boost-v2-eagle-import #SUPPLY?
 U 1 1 5ECBF78C
 P 10550 3750
@@
 $EndComp
 $Comp
-L PowerBoard-Boost-v2-eagle-import:GND #GND?
+L PowerBoth-rescue:GND-PowerBoard-Boost-v2-eagle-import #GND?
 U 1 1 5ECBF792
 P 8550 3150
@@
 $EndComp
 $Comp
-L PowerBoard-Boost-v2-eagle-import:TEST_POINTROUND-1MM TP?
+L PowerBoth-rescue:TEST_POINTROUND-1MM-PowerBoard-Boost-v2-eagle-import TP?
 U 1 1 5ECBF798
 P 950 1750
@@
 $EndComp
 $Comp
-L PowerBoard-Boost-v2-eagle-import:2X10-2MMSMD J?
+L PowerBoth-rescue:2X10-2MMSMD-PowerBoard-Boost-v2-eagle-import J?
 U 1 1 5ECBF79E
 P 9400 1650
@@
 $EndComp
 $Comp
-L PowerBoard-Boost-v2-eagle-import:5V #SUPPLY?
+L PowerBoth-rescue:5V-PowerBoard-Boost-v2-eagle-import #SUPPLY?
 U 1 1 5ECBF7A4
 P 9700 1150
@@
 $EndComp
 $Comp
-L PowerBoard-Boost-v2-eagle-import:GND #GND?
+L PowerBoth-rescue:GND-PowerBoard-Boost-v2-eagle-import #GND?
 U 1 1 5ECBF7AA
 P 9700 2050
@@
 $EndComp
 $Comp
-L PowerBoard-Boost-v2-eagle-import:TEST_POINTROUND-1MM TP2-STAT?
+L PowerBoth-rescue:TEST_POINTROUND-1MM-PowerBoard-Boost-v2-eagle-import TP2-STAT?
 U 1 1 5ECBF7B0
 P 2550 1650

Commit message: Replacing the SEPIC converter.
Parts:
- removed J302: 2X10-2MMSMD, PowerBoard-Boost-v2:2X10-2MM, symbol PowerBoth-rescue:2X10-2MMSMD-PowerBoard-Boost-v2-eagle-import
Connections:
- net labels removed: CHG_CON, VBATT
- wire segments 111 -> 80
- no-connect marks 2 -> 0
Changed lines of the file:
@@
 $Descr A4 11693 8268
 encoding utf-8
-Sheet 3 3
+Sheet 3 5
 Title ""
 Date ""
@@
 GND
 Wire Wire Line
-	9500 1750 9500 1850
-Wire Wire Line
-	9500 1850 9600 1850
-Wire Wire Line
-	9600 1850 9700 1850
-Wire Wire Line
-	9700 1850 9700 1950
-Wire Wire Line
-	9600 1750 9600 1850
-Wire Wire Line
-	9700 1750 9700 1850
-Wire Wire Line
-	9800 1750 9800 1850
-Wire Wire Line
-	9800 1850 9700 1850
-Wire Wire Line
-	9800 1850 9900 1850
-Wire Wire Line
-	9900 1850 9900 1750
-Wire Wire Line
-	9900 1850 10000 1850
-Wire Wire Line
-	10000 1850 10000 1750
-Wire Wire Line
-	10000 1850 10100 1850
-Wire Wire Line
-	10100 1850 10100 1750
-Wire Wire Line
-	10100 1850 10200 1850
-Wire Wire Line
-	10200 1850 10200 1750
-Connection ~ 9600 1850
-Connection ~ 9700 1850
-Connection ~ 9800 1850
-Connection ~ 9900 1850
-Connection ~ 10000 1850
-Connection ~ 10100 1850
-Wire Wire Line
-	10400 1350 10400 1050
-Wire Wire Line
 	2050 5200 1650 5200
 Wire Wire Line
@@
 Text Label 8850 4050 0    10   ~ 0
 5V
-Wire Wire Line
-	9500 1350 9500 1250
-Wire Wire Line
-	9500 1250 9600 1250
-Wire Wire Line
-	9600 1250 9700 1250
-Wire Wire Line
-	9700 1250 9700 1150
-Wire Wire Line
-	9600 1350 9600 1250
-Wire Wire Line
-	9700 1350 9700 1250
-Wire Wire Line
-	9800 1350 9800 1250
-Wire Wire Line
-	9800 1250 9700 1250
-Wire Wire Line
-	9900 1350 9900 1250
-Wire Wire Line
-	9900 1250 9800 1250
-Wire Wire Line
-	10000 1350 10000 1250
-Wire Wire Line
-	10000 1250 9900 1250
-Wire Wire Line
-	10100 1350 10100 1250
-Wire Wire Line
-	10100 1250 10000 1250
-Connection ~ 9600 1250
-Connection ~ 9700 1250
-Connection ~ 9800 1250
-Connection ~ 9900 1250
-Connection ~ 10000 1250
 $Comp
 L PowerBoth-rescue:LM3488QMM_NOPBDGK8-M-PowerBoard-Boost-v2-eagle-import U?
@@
 $EndComp
 $Comp
-L PowerBoth-rescue:2X10-2MMSMD-PowerBoard-Boost-v2-eagle-import J?
-U 1 1 5ECBF79E
-P 9400 1650
-AR Path="/5ECBF79E" Ref="J?"  Part="1"
-AR Path="/5E8AAE5F/5ECBF79E" Ref="J?"  Part="1"
-AR Path="/5ECA2372/5E8AAE5F/5ECBF79E" Ref="J?"  Part="1"
-AR Path="/5ECA2372/5ECBF79E" Ref="J302"  Part="1"
-F 0 "J302" H 10500 1750 59  0000 L BNN
-F 1 "2X10-2MMSMD" H 10500 1650 59  0000 L BNN
-F 2 "PowerBoard-Boost-v2:2X10-2MM" H 9400 1650 50  0001 C CNN
-F 3 "" H 9400 1650 50  0001 C CNN
-	1    9400 1650
-	1    0    0    -1
-$EndComp
-$Comp
-L PowerBoth-rescue:5V-PowerBoard-Boost-v2-eagle-import #SUPPLY?
-U 1 1 5ECBF7A4
-P 9700 1150
-AR Path="/5ECBF7A4" Ref="#SUPPLY?"  Part="1"
-AR Path="/5E8AAE5F/5ECBF7A4" Ref="#SUPPLY?"  Part="1"
-AR Path="/5ECA2372/5E8AAE5F/5ECBF7A4" Ref="#SUPPLY?"  Part="1"
-AR Path="/5ECA2372/5ECBF7A4" Ref="#SUPPLY0302"  Part="1"
-F 0 "#SUPPLY0302" H 9700 1150 50  0001 C CNN
-F 1 "5V" H 9700 1260 59  0000 C BNN
-F 2 "" H 9700 1150 50  0001 C CNN
-F 3 "" H 9700 1150 50  0001 C CNN
-	1    9700 1150
-	1    0    0    -1
-$EndComp
-$Comp
-L PowerBoth-rescue:GND-PowerBoard-Boost-v2-eagle-import #GND?
-U 1 1 5ECBF7AA
-P 9700 2050
-AR Path="/5ECBF7AA" Ref="#GND?"  Part="1"
-AR Path="/5E8AAE5F/5ECBF7AA" Ref="#GND?"  Part="1"
-AR Path="/5ECA2372/5E8AAE5F/5ECBF7AA" Ref="#GND?"  Part="1"
-AR Path="/5ECA2372/5ECBF7AA" Ref="#GND0307"  Part="1"
-F 0 "#GND0307" H 9700 2050 50  0001 C CNN
-F 1 "GND" H 9600 1950 59  0000 L BNN
-F 2 "" H 9700 2050 50  0001 C CNN
-F 3 "" H 9700 2050 50  0001 C CNN
-	1    9700 2050
-	1    0    0    -1
-$EndComp
-$Comp
 L PowerBoth-rescue:TEST_POINTROUND-1MM-PowerBoard-Boost-v2-eagle-import TP2-STAT?
 U 1 1 5ECBF7B0
@@
 Text HLabel 2550 1650 3    39   Input ~ 0
 CHSTAT
-Text HLabel 10400 1050 1    39   Input ~ 0
-CHG_CON
 Text HLabel 950  1750 3    39   Input ~ 0
 V+CH
@@
 Text HLabel 7450 3350 0    39   Input ~ 0
 V+ToBoost
-Text HLabel 10400 1750 3    39   Input ~ 0
-CHSTAT
-Text HLabel 10300 1750 3    39   Input ~ 0
-VBATT
-NoConn ~ 10300 1350
-NoConn ~ 10200 1350
 $Comp
 L power:PWR_FLAG #FLG0102
@@
 	1    0    0    -1
 $EndComp
-$Comp
-L power:PWR_FLAG #FLG0103
-U 1 1 5E923499
-P 9900 1250
-F 0 "#FLG0103" H 9900 1325 50  0001 C CNN
-F 1 "PWR_FLAG" H 9900 1423 50  0000 C CNN
-F 2 "" H 9900 1250 50  0001 C CNN
-F 3 "~" H 9900 1250 50  0001 C CNN
-	1    9900 1250
-	1    0    0    -1
-$EndComp

Commit message: Replacing the SEPIC converter.
Parts:
- CBP301: footprint PowerBoard-Boost-v2:C1206 -> Capacitor_SMD:C_1206_3216Metric_Pad1.42x1.75mm_HandSolder
Changed lines of the file:
@@
 F 0 "CBP301" H 2590 6125 59  0000 L BNN
 F 1 "0.1uF" H 2590 5935 59  0000 L BNN
-F 2 "PowerBoard-Boost-v2:C1206" H 2550 6100 50  0001 C CNN
+F 2 "Capacitor_SMD:C_1206_3216Metric_Pad1.42x1.75mm_HandSolder" H 2550 6100 50  0001 C CNN
 F 3 "" H 2550 6100 50  0001 C CNN
 	1    2550 6100
