File: PowerBoard/Charger/PowerBoard.sch (KiCad schematic (older format))
At the start: 19 parts, among them J201 PJ-079AH, J202 2MM-1X5, M201 IRF7205, Q201 IRF7205, U201 LTC4002ES8-4.2PBFSO-8_S-M

Commit message: Cleanup to assemble the power board V2.
Parts:
- C201, C202, C203: symbol PowerBoard-eagle-import:C-USC1210 -> PowerBoth-rescue:C-USC1210-PowerBoard-eagle-import
- CC201: symbol PowerBoard-eagle-import:C-USC0603 -> PowerBoth-rescue:C-USC0603-PowerBoard-eagle-import
- D201, D202, D203: symbol PowerBoard-eagle-import:B330A-13 -> PowerBoth-rescue:B330A-13-PowerBoard-eagle-import
- J201: symbol PowerBoard-eagle-import:PJ-079AH -> PowerBoth-rescue:PJ-079AH-PowerBoard-eagle-import
- J202: symbol PowerBoard-eagle-import:2MM-1X5 -> PowerBoth-rescue:2MM-1X5-PowerBoard-eagle-import
- L201: symbol PowerBoard-eagle-import:B952AS-H-220M=P3 -> PowerBoth-rescue:B952AS-H-220M=P3-PowerBoard-eagle-import
- M201, Q201: symbol PowerBoard-eagle-import:IRF7205 -> PowerBoth-rescue:IRF7205-PowerBoard-eagle-import
- R201, RC201, RSENSE201: symbol PowerBoard-eagle-import:R-US_R1206 -> PowerBoth-rescue:R-US_R1206-PowerBoard-eagle-import
- R202: symbol PowerBoard-eagle-import:RESISTOR1206 -> PowerBoth-rescue:RESISTOR1206-PowerBoard-eagle-import
- TP201, TP202: symbol PowerBoard-eagle-import:TEST_POINTROUND-1MM -> PowerBoth-rescue:TEST_POINTROUND-1MM-PowerBoard-eagle-import
- U201: symbol PowerBoard-eagle-import:LTC4002ES8-4.2PBFSO-8_S-M -> PowerBoth-rescue:LTC4002ES8-4.2PBFSO-8_S-M-PowerBoard-eagle-import
Changed lines of the file:
@@
 Connection ~ 8800 4500
 $Comp
-L PowerBoard-eagle-import:2MM-1X5 J202
+L PowerBoth-rescue:2MM-1X5-PowerBoard-eagle-import J202
 U 1 1 449C7C68
 P 5900 5200
@@
 $EndComp
 $Comp
-L PowerBoard-eagle-import:LTC4002ES8-4.2PBFSO-8_S-M U201
+L PowerBoth-rescue:LTC4002ES8-4.2PBFSO-8_S-M-PowerBoard-eagle-import U201
 U 1 1 94FABF20
 P 3900 3900
@@
 $EndComp
 $Comp
-L PowerBoard-eagle-import:IRF7205 M201
+L PowerBoth-rescue:IRF7205-PowerBoard-eagle-import M201
 U 1 1 63C736F8
 P 3600 4200
@@
 $EndComp
 $Comp
-L PowerBoard-eagle-import:B952AS-H-220M=P3 L201
+L PowerBoth-rescue:B952AS-H-220M=P3-PowerBoard-eagle-import L201
 U 1 1 737D6DDD
 P 3600 5000
@@
 $EndComp
 $Comp
-L PowerBoard-eagle-import:B330A-13 D201
+L PowerBoth-rescue:B330A-13-PowerBoard-eagle-import D201
 U 1 1 C78C3FBD
 P 2500 3400
@@
 $EndComp
 $Comp
-L PowerBoard-eagle-import:B330A-13 D202
+L PowerBoth-rescue:B330A-13-PowerBoard-eagle-import D202
 U 1 1 0CADE672
 P 3800 4900
@@
 $EndComp
 $Comp
-L PowerBoard-eagle-import:GND #GND0202
+L PowerBoth-rescue:GND-PowerBoard-eagle-import #GND0202
 U 1 1 8DA2BB24
 P 4000 5200
@@
 $EndComp
 $Comp
-L PowerBoard-eagle-import:R-US_R1206 RSENSE201
+L PowerBoth-rescue:R-US_R1206-PowerBoard-eagle-import RSENSE201
 U 1 1 6ED65E17
 P 6800 4100
@@
 $EndComp
 $Comp
-L PowerBoard-eagle-import:GND #GND0204
+L PowerBoth-rescue:GND-PowerBoard-eagle-import #GND0204
 U 1 1 4877C9E2
 P 6500 5400
@@
 $EndComp
 $Comp
-L PowerBoard-eagle-import:C-USC1210 C202
+L PowerBoth-rescue:C-USC1210-PowerBoard-eagle-import C202
 U 1 1 E7D47EA7
 P 3300 3700
@@
 $EndComp
 $Comp
-L PowerBoard-eagle-import:C-USC1210 C203
+L PowerBoth-rescue:C-USC1210-PowerBoard-eagle-import C203
 U 1 1 483159C7
 P 6800 5000
@@
 $EndComp
 $Comp
-L PowerBoard-eagle-import:C-USC1210 C201
+L PowerBoth-rescue:C-USC1210-PowerBoard-eagle-import C201
 U 1 1 88676885
 P 3000 3700
@@
 $EndComp
 $Comp
-L PowerBoard-eagle-import:C-USC0603 CC201
+L PowerBoth-rescue:C-USC0603-PowerBoard-eagle-import CC201
 U 1 1 7170E37A
 P 4100 3100
@@
 $EndComp
 $Comp
-L PowerBoard-eagle-import:GND #GND0201
+L PowerBoth-rescue:GND-PowerBoard-eagle-import #GND0201
 U 1 1 21137572
 P 3000 4300
@@
 $EndComp
 $Comp
-L PowerBoard-eagle-import:GND #GND0203
+L PowerBoth-rescue:GND-PowerBoard-eagle-import #GND0203
 U 1 1 12C122FD
 P 4900 3300
@@
 $EndComp
 $Comp
-L PowerBoard-eagle-import:R-US_R1206 RC201
+L PowerBoth-rescue:R-US_R1206-PowerBoard-eagle-import RC201
 U 1 1 F7D68A95
 P 4600 3100
@@
 $EndComp
 $Comp
-L PowerBoard-eagle-import:R-US_R1206 R201
+L PowerBoth-rescue:R-US_R1206-PowerBoard-eagle-import R201
 U 1 1 B6BC5140
 P 5300 4700
@@
 $EndComp
 $Comp
-L PowerBoard-eagle-import:RESISTOR1206 R202
+L PowerBoth-rescue:RESISTOR1206-PowerBoard-eagle-import R202
 U 1 1 A3C89E4B
 P 8400 3600
@@
 $EndComp
 $Comp
-L PowerBoard-eagle-import:GND #GND0205
+L PowerBoth-rescue:GND-PowerBoard-eagle-import #GND0205
 U 1 1 FF2A2D77
 P 8800 3900
@@
 $EndComp
 $Comp
-L PowerBoard-eagle-import:IRF7205 Q201
+L PowerBoth-rescue:IRF7205-PowerBoard-eagle-import Q201
 U 1 1 E6D570CA
 P 8100 4300
@@
 $EndComp
 $Comp
-L PowerBoard-eagle-import:PJ-079AH J201
+L PowerBoth-rescue:PJ-079AH-PowerBoard-eagle-import J201
 U 1 1 C3E76336
 P 1800 3600
@@
 $EndComp
 $Comp
-L PowerBoard-eagle-import:B330A-13 D203
+L PowerBoth-rescue:B330A-13-PowerBoard-eagle-import D203
 U 1 1 93886C31
 P 8400 4100
@@
 $EndComp
 $Comp
-L PowerBoard-eagle-import:TEST_POINTROUND-1MM TP201
+L PowerBoth-rescue:TEST_POINTROUND-1MM-PowerBoard-eagle-import TP201
 U 1 1 0B1FCAED
 P 5000 4900
@@
 Load sharing circuit.\nBased on Microchip\nApplication Note AN1149.
 $Comp
-L PowerBoard-eagle-import:TEST_POINTROUND-1MM TP202
+L PowerBoth-rescue:TEST_POINTROUND-1MM-PowerBoard-eagle-import TP202
 U 1 1 5E932987
 P 7350 3400

Commit message: Add display circuitry.
Changed lines of the file:
@@
 	2500 4000 3000 4000
 Connection ~ 3000 4000
-Text Label 3000 3900 0    10   ~ 0
-GND
 Wire Wire Line
 	4800 3100 4900 3100

Commit message: Replacing the SEPIC converter.
Parts:
- removed D203: B330A-13, PowerBoard:SMA-M, symbol PowerBoth-rescue:B330A-13-PowerBoard-eagle-import
- removed Q201: IRF7205, PowerBoard:8SOIC, symbol PowerBoth-rescue:IRF7205-PowerBoard-eagle-import
- removed R202: 56K, PowerBoard:1206, symbol PowerBoth-rescue:RESISTOR1206-PowerBoard-eagle-import
Connections:
- net labels removed: V+ToBoost, VCC
- wire segments 83 -> 67
Other:
- note removed: "Load sharing circuit.\nBased on Microchip\nApplication Note AN1149."
Changed lines of the file:
@@
 $Descr A4 11693 8268
 encoding utf-8
-Sheet 2 3
+Sheet 2 5
 Title ""
 Date ""
@@
 Connection ~ 2400 3400
 Wire Wire Line
-	8100 4000 8100 3600
-Wire Wire Line
-	8100 3600 8100 3500
-Wire Wire Line
-	8100 4000 8200 4000
-Wire Wire Line
-	8100 3600 8200 3600
-Wire Wire Line
-	8200 4100 8200 4000
-Wire Wire Line
-	8400 4100 8400 4000
-Wire Wire Line
-	8400 4000 8200 4000
-Connection ~ 8100 3600
-Connection ~ 8200 4000
-Text Label 8100 4000 0    10   ~ 0
-VCC
-Wire Wire Line
 	2900 3400 3000 3400
 Wire Wire Line
@@
 	4900 3100 4900 3200
 Wire Wire Line
-	8600 3600 8800 3600
-Wire Wire Line
-	8800 3600 8800 3800
-Text Label 8600 3600 0    10   ~ 0
-GND
-Wire Wire Line
 	3600 4400 3600 4500
 Wire Wire Line
@@
 Wire Wire Line
 	7400 4500 6800 4500
-Wire Wire Line
-	7900 4500 7900 4300
-Wire Wire Line
-	7900 4500 7400 4500
 Connection ~ 6800 4300
 Connection ~ 6800 4700
 Connection ~ 6800 4800
 Connection ~ 6800 4500
-Connection ~ 7400 4500
-Wire Wire Line
-	8300 4300 8400 4300
-Wire Wire Line
-	8400 4300 8400 4500
-Wire Wire Line
-	8400 4500 8800 4500
-Wire Wire Line
-	8800 4100 8800 4500
-Wire Wire Line
-	8800 4500 9600 4500
-Connection ~ 8800 4500
 $Comp
 L PowerBoth-rescue:2MM-1X5-PowerBoard-eagle-import J202
@@
 $Comp
 L PowerBoth-rescue:B952AS-H-220M=P3-PowerBoard-eagle-import L201
-U 1 1 737D6DDD
+U 1 1 5ED47BE7
 P 3600 5000
 F 0 "L201" H 3564 5132 116 0000 L BNN
@@
 $Comp
 L PowerBoth-rescue:C-USC1210-PowerBoard-eagle-import C202
-U 1 1 E7D47EA7
+U 1 1 5ED47BE6
 P 3300 3700
 F 0 "C202" H 3340 3725 59  0000 L BNN
@@
 $EndComp
 $Comp
-L PowerBoth-rescue:RESISTOR1206-PowerBoard-eagle-import R202
-U 1 1 A3C89E4B
-P 8400 3600
-F 0 "R202" H 8250 3659 59  0000 L BNN
-F 1 "56K" H 8250 3470 59  0000 L BNN
-F 2 "PowerBoard:1206" H 8400 3600 50  0001 C CNN
-F 3 "" H 8400 3600 50  0001 C CNN
-	1    8400 3600
-	-1   0    0    1
-$EndComp
-$Comp
-L PowerBoth-rescue:GND-PowerBoard-eagle-import #GND0205
-U 1 1 FF2A2D77
-P 8800 3900
-F 0 "#GND0205" H 8800 3900 50  0001 C CNN
-F 1 "GND" H 8700 3800 59  0000 L BNN
-F 2 "" H 8800 3900 50  0001 C CNN
-F 3 "" H 8800 3900 50  0001 C CNN
-	1    8800 3900
-	1    0    0    -1
-$EndComp
-$Comp
-L PowerBoth-rescue:IRF7205-PowerBoard-eagle-import Q201
-U 1 1 E6D570CA
-P 8100 4300
-F 0 "Q201" H 7750 4150 59  0000 L TNN
-F 1 "IRF7205" V 8260 4480 59  0000 L TNN
-F 2 "PowerBoard:8SOIC" H 8100 4300 50  0001 C CNN
-F 3 "" H 8100 4300 50  0001 C CNN
-F 4 "C55419" H 8100 4300 50  0001 C CNN "LCSC Part Number"
-	1    8100 4300
-	0    -1   1    0
-$EndComp
-$Comp
 L PowerBoth-rescue:PJ-079AH-PowerBoard-eagle-import J201
 U 1 1 C3E76336
@@
 	1    1800 3600
 	1    0    0    -1
-$EndComp
-$Comp
-L PowerBoth-rescue:B330A-13-PowerBoard-eagle-import D203
-U 1 1 93886C31
-P 8400 4100
-F 0 "D203" H 8500 4306 116 0000 L BNN
-F 1 "B330A-13" H 8500 4182 116 0000 L BNN
-F 2 "PowerBoard:SMA-M" H 8400 4100 50  0001 C CNN
-F 3 "" H 8400 4100 50  0001 C CNN
-	1    8400 4100
-	0    1    1    0
 $EndComp
 $Comp
@@
 	-1   0    0    1
 $EndComp
-Wire Notes Line
-	7800 3200 9000 3200
-Wire Notes Line
-	9000 3200 9000 5500
-Wire Notes Line
-	9000 5500 7800 5500
-Wire Notes Line
-	7800 5500 7800 3200
-Text Notes 7850 5450 0    47   ~ 0
-Load sharing circuit.\nBased on Microchip\nApplication Note AN1149.
 $Comp
 L PowerBoth-rescue:TEST_POINTROUND-1MM-PowerBoard-eagle-import TP202
@@
 Wire Wire Line
 	7400 3400 7400 4500
-Text HLabel 9600 4500 2    39   Input ~ 0
-V+ToBoost
 Text HLabel 2300 3500 2    39   Input ~ 0
 CHG_CON
 Text HLabel 2400 2700 1    39   Input ~ 0
 V+CH
-Text HLabel 8100 3500 1    39   Input ~ 0
-V+CH
 Text HLabel 5000 4900 0    39   Input ~ 0

Commit message: Replacing the SEPIC converter.
Parts:
- C201: footprint PowerBoard:C1210 -> Capacitor_SMD:C_0805_2012Metric_Pad1.15x1.40mm_HandSolder
- C202, C203: footprint PowerBoard:C1210 -> Capacitor_SMD:C_1210_3225Metric_Pad1.42x2.65mm_HandSolder
- CC201: footprint PowerBoard:C0603 -> Capacitor_SMD:C_0603_1608Metric_Pad1.05x0.95mm_HandSolder
Changed lines of the file:
@@
 F 0 "C202" H 3340 3725 59  0000 L BNN
 F 1 "10uF" H 3340 3535 59  0000 L BNN
-F 2 "PowerBoard:C1210" H 3300 3700 50  0001 C CNN
+F 2 "Capacitor_SMD:C_1210_3225Metric_Pad1.42x2.65mm_HandSolder" H 3300 3700 50  0001 C CNN
 F 3 "" H 3300 3700 50  0001 C CNN
 	1    3300 3700
@@
 F 0 "C203" H 6840 5025 59  0000 L BNN
 F 1 "22uF" H 6840 4835 59  0000 L BNN
-F 2 "PowerBoard:C1210" H 6800 5000 50  0001 C CNN
+F 2 "Capacitor_SMD:C_1210_3225Metric_Pad1.42x2.65mm_HandSolder" H 6800 5000 50  0001 C CNN
 F 3 "" H 6800 5000 50  0001 C CNN
 	1    6800 5000
@@
 F 0 "C201" H 3040 3725 59  0000 L BNN
 F 1 "0.1uF" H 3040 3535 59  0000 L BNN
-F 2 "PowerBoard:C1210" H 3000 3700 50  0001 C CNN
+F 2 "Capacitor_SMD:C_0805_2012Metric_Pad1.15x1.40mm_HandSolder" H 3000 3700 50  0001 C CNN
 F 3 "" H 3000 3700 50  0001 C CNN
 F 4 "1" H 3000 3700 50  0001 C CNN "LCSC Part Number"
@@
 F 0 "CC201" H 4140 3125 59  0000 L BNN
 F 1 "0.47uF" H 4140 2935 59  0000 L BNN
-F 2 "PowerBoard:C0603" H 4100 3100 50  0001 C CNN
+F 2 "Capacitor_SMD:C_0603_1608Metric_Pad1.05x0.95mm_HandSolder" H 4100 3100 50  0001 C CNN
 F 3 "" H 4100 3100 50  0001 C CNN
 	1    4100 3100

Commit message: Separating the power board branch.
Parts:
- removed R201: 2K, PowerBoard:R1206, symbol PowerBoth-rescue:R-US_R1206-PowerBoard-eagle-import
- removed TP201, TP202: TEST_POINTROUND-1MM, PowerBoard:TEST_POINT_ROUND_1MM, symbol PowerBoth-rescue:TEST_POINTROUND-1MM-PowerBoard-eagle-import
- C201: DigiKey (none) -> C0805C104M3RACTU; LCSC Part Number 1 -> C49678
- C202: footprint Capacitor_SMD:C_1210_3225Metric_Pad1.42x2.65mm_HandSolder -> Capacitor_SMD:C_0805_2012Metric_Pad1.15x1.40mm_HandSolder; DigiKey (none) -> EMK212BB7106MG-T; LCSC Part Number (none) -> C15850
- C203: DigiKey (none) -> CL21A226MAQNNNE; LCSC Part Number (none) -> C45783
- CC201: DigiKey (none) -> C0805C474K3RACAUTO
- D201, D202: DigiKey (none) -> B330B-13-F; LCSC Part Number (none) -> C110485
- J201: DigiKey (none) -> PJ-079AH
- J202: DigiKey (none) -> 0533250560
- L201: DigiKey (none) -> #B952AS-H-6R8N=P3
- M201: DigiKey (none) -> IRF7205TRPBF
- RC201: value R-US_R1206 -> 2.2K; DigiKey (none) -> RC0805FR-072K2L
- RSENSE201: DigiKey (none) -> KDV08FR068ET
- U201: DigiKey (none) -> LTC4002ES8-4.2#TRPBF
Connections:
- wire segments 67 -> 64
Changed lines of the file:
@@
 $Descr A4 11693 8268
 encoding utf-8
-Sheet 2 5
+Sheet 2 4
 Title ""
 Date ""
@@
 	4400 3100 4300 3100
 Wire Wire Line
-	5500 4700 5700 4700
-Wire Wire Line
 	5700 4700 5700 4500
 Wire Wire Line
@@
 Wire Wire Line
 	6200 4500 6200 4200
-Wire Wire Line
-	5100 4700 5000 4700
 Wire Wire Line
 	5000 4900 5000 4700
@@
 F 2 "PowerBoard:2MM_1X5" H 5900 5200 50  0001 C CNN
 F 3 "" H 5900 5200 50  0001 C CNN
+F 4 "0533250560" H 5900 5200 50  0001 C CNN "DigiKey"
 	1    5900 5200
 	0    1    -1   0
@@
 F 2 "PowerBoard:SO-8_S-M" H 3900 3900 50  0001 C CNN
 F 3 "" H 3900 3900 50  0001 C CNN
+F 4 "LTC4002ES8-4.2#TRPBF" H 3900 3900 50  0001 C CNN "DigiKey"
 	1    3900 3900
 	1    0    0    -1
@@
 F 3 "" H 3600 4200 50  0001 C CNN
 F 4 "C55419" H 3600 4200 50  0001 C CNN "LCSC Part Number"
+F 5 "IRF7205TRPBF" H 3600 4200 50  0001 C CNN "DigiKey"
 	1    3600 4200
 	-1   0    0    1
@@
 F 2 "PowerBoard:IND_B952AS-H-220M=P3" H 3600 5000 50  0001 C CNN
 F 3 "" H 3600 5000 50  0001 C CNN
+F 4 "#B952AS-H-6R8N=P3" H 3600 5000 50  0001 C CNN "DigiKey"
 	1    3600 5000
 	0    1    1    0
@@
 F 2 "PowerBoard:SMA-M" H 2500 3400 50  0001 C CNN
 F 3 "" H 2500 3400 50  0001 C CNN
+F 4 "B330B-13-F" H 2500 3400 50  0001 C CNN "DigiKey"
+F 5 "C110485" H 2500 3400 50  0001 C CNN "LCSC Part Number"
 	1    2500 3400
 	0    1    1    0
@@
 F 2 "PowerBoard:SMA-M" H 3800 4900 50  0001 C CNN
 F 3 "" H 3800 4900 50  0001 C CNN
+F 4 "B330B-13-F" H 3800 4900 50  0001 C CNN "DigiKey"
+F 5 "C110485" H 3800 4900 50  0001 C CNN "LCSC Part Number"
 	1    3800 4900
 	1    0    0    -1
@@
 F 2 "PowerBoard:R1206" H 6800 4100 50  0001 C CNN
 F 3 "" H 6800 4100 50  0001 C CNN
+F 4 "KDV08FR068ET" H 6800 4100 50  0001 C CNN "DigiKey"
 	1    6800 4100
 	0    -1   -1   0
@@
 F 0 "C202" H 3340 3725 59  0000 L BNN
 F 1 "10uF" H 3340 3535 59  0000 L BNN
-F 2 "Capacitor_SMD:C_1210_3225Metric_Pad1.42x2.65mm_HandSolder" H 3300 3700 50  0001 C CNN
+F 2 "Capacitor_SMD:C_0805_2012Metric_Pad1.15x1.40mm_HandSolder" H 3300 3700 50  0001 C CNN
 F 3 "" H 3300 3700 50  0001 C CNN
+F 4 "EMK212BB7106MG-T" H 3300 3700 50  0001 C CNN "DigiKey"
+F 5 "C15850" H 3300 3700 50  0001 C CNN "LCSC Part Number"
 	1    3300 3700
 	1    0    0    -1
@@
 F 2 "Capacitor_SMD:C_1210_3225Metric_Pad1.42x2.65mm_HandSolder" H 6800 5000 50  0001 C CNN
 F 3 "" H 6800 5000 50  0001 C CNN
+F 4 "CL21A226MAQNNNE" H 6800 5000 50  0001 C CNN "DigiKey"
+F 5 "C45783" H 6800 5000 50  0001 C CNN "LCSC Part Number"
 	1    6800 5000
 	1    0    0    -1
@@
 F 2 "Capacitor_SMD:C_0805_2012Metric_Pad1.15x1.40mm_HandSolder" H 3000 3700 50  0001 C CNN
 F 3 "" H 3000 3700 50  0001 C CNN
-F 4 "1" H 3000 3700 50  0001 C CNN "LCSC Part Number"
+F 4 "C49678" H 3000 3700 50  0001 C CNN "LCSC Part Number"
+F 5 "C0805C104M3RACTU" H 3000 3700 50  0001 C CNN "DigiKey"
 	1    3000 3700
 	1    0    0    -1
@@
 F 2 "Capacitor_SMD:C_0603_1608Metric_Pad1.05x0.95mm_HandSolder" H 4100 3100 50  0001 C CNN
 F 3 "" H 4100 3100 50  0001 C CNN
+F 4 "C0805C474K3RACAUTO" H 4100 3100 50  0001 C CNN "DigiKey"
 	1    4100 3100
 	0    -1   -1   0
@@
 P 4600 3100
 F 0 "RC201" H 4450 3159 59  0000 L BNN
-F 1 "R-US_R1206" H 4450 2970 59  0000 L BNN
+F 1 "2.2K" H 4450 2970 59  0000 L BNN
 F 2 "PowerBoard:R1206" H 4600 3100 50  0001 C CNN
 F 3 "" H 4600 3100 50  0001 C CNN
+F 4 "RC0805FR-072K2L" H 4600 3100 50  0001 C CNN "DigiKey"
 	1    4600 3100
-	-1   0    0    1
-$EndComp
-$Comp
-L PowerBoth-rescue:R-US_R1206-PowerBoard-eagle-import R201
-U 1 1 B6BC5140
-P 5300 4700
-F 0 "R201" H 5150 4759 59  0000 L BNN
-F 1 "2K" H 5150 4570 59  0000 L BNN
-F 2 "PowerBoard:R1206" H 5300 4700 50  0001 C CNN
-F 3 "" H 5300 4700 50  0001 C CNN
-	1    5300 4700
 	-1   0    0    1
 $EndComp
@@
 F 2 "PowerBoard:CUI_PJ-079AH" H 1800 3600 50  0001 C CNN
 F 3 "" H 1800 3600 50  0001 C CNN
+F 4 "PJ-079AH" H 1800 3600 50  0001 C CNN "DigiKey"
 	1    1800 3600
 	1    0    0    -1
 $EndComp
-$Comp
-L PowerBoth-rescue:TEST_POINTROUND-1MM-PowerBoard-eagle-import TP201
-U 1 1 0B1FCAED
-P 5000 4900
-F 0 "TP201" H 4900 5200 42  0000 L BNN
-F 1 "TEST_POINTROUND-1MM" V 4900 4900 42  0000 L BNN
-F 2 "PowerBoard:TEST_POINT_ROUND_1MM" H 5000 4900 50  0001 C CNN
-F 3 "" H 5000 4900 50  0001 C CNN
-	1    5000 4900
-	-1   0    0    1
-$EndComp
-$Comp
-L PowerBoth-rescue:TEST_POINTROUND-1MM-PowerBoard-eagle-import TP202
-U 1 1 5E932987
-P 7350 3400
-F 0 "TP202" H 7250 3700 42  0000 L BNN
-F 1 "TEST_POINTROUND-1MM" V 7250 3400 42  0000 L BNN
-F 2 "PowerBoard:TEST_POINT_ROUND_1MM" H 7350 3400 50  0001 C CNN
-F 3 "" H 7350 3400 50  0001 C CNN
-	1    7350 3400
-	0    -1   -1   0
-$EndComp
-Wire Wire Line
-	7350 3400 7400 3400
-Connection ~ 7400 3400
-Wire Wire Line
-	7400 3400 7400 4500
 Text HLabel 2300 3500 2    39   Input ~ 0
 CHG_CON
@@
 Text HLabel 7400 2900 1    39   Input ~ 0
 VBATT
-Wire Wire Line
-	7400 2900 7400 3400
 $Comp
 L power:PWR_FLAG #FLG0101
@@
 $EndComp
 Connection ~ 3700 3400
+Wire Wire Line
+	5000 4700 5700 4700
+Wire Wire Line
+	7400 2900 7400 4500
 $EndSCHEMATC
