File: CPU/CPU.sch (KiCad schematic (older format))
At the start: 13 parts, among them J101 Conn_02x10_Odd_Even, J102 Conn_02x14_Odd_Even_MountingP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, Q101 IRLML0040TR, Q102 IRLML0040TR, SW101 SW_SPDT

Commit message: Corrected the issues with v1 of the CPU board. Moved to 0.8mm board. Should be ready for another order.
Parts:
- removed C101: 47uF, Capacitor_SMD:C_0805_2012Metric_Pad1.15x1.40mm_HandSolder, symbol Device:C
- removed TP102: TestPoint, TestPoint:TestPoint_Pad_D1.0mm, symbol Connector:TestPoint
- Pi101: footprint CPU:RASPBERRYPI_Zero-No_Mounting_Holes -> CPU:RASPBERRYPI_Zero-No_Mounting_Holes_SMD_Flat
Connections:
- net labels removed: TGUARD
- wire segments 107 -> 102
- no-connect marks 18 -> 29
Changed lines of the file:
@@
 F 0 "Pi101" H 3150 7600 50  0000 L BNN
 F 1 "RPI-ZERO" H 3150 7525 50  0000 L BNN
-F 2 "CPU:RASPBERRYPI_Zero-No_Mounting_Holes" H 3950 6200 50  0001 C CNN
+F 2 "CPU:RASPBERRYPI_Zero-No_Mounting_Holes_SMD_Flat" H 3950 6200 50  0001 C CNN
 F 3 "" H 3950 6200 50  0001 C CNN
 	1    3950 6200
@@
 $EndComp
 $Comp
-L power:+3V3 #PWR0102
-U 1 1 5E97A3AA
-P 2950 4950
-F 0 "#PWR0102" H 2950 4800 50  0001 C CNN
-F 1 "+3V3" H 2965 5123 50  0000 C CNN
-F 2 "" H 2950 4950 50  0001 C CNN
-F 3 "" H 2950 4950 50  0001 C CNN
-	1    2950 4950
-	1    0    0    -1
-$EndComp
-Wire Wire Line
-	3050 5000 2950 5000
-Wire Wire Line
-	2950 5000 2950 4950
-$Comp
 L CPU-eagle-import:GND #GND0102
 U 1 1 5E988321
@@
 Connection ~ 2550 6200
 Wire Wire Line
-	2950 5000 2950 5800
-Wire Wire Line
 	2950 5800 3050 5800
-Connection ~ 2950 5000
 $Comp
 L CPU-eagle-import:GND #GND0105
@@
 	3500 2900 3400 2900
 Connection ~ 3500 2900
-Text Label 3600 3200 2    39   ~ 0
-Pi7
-Text Label 3600 3400 2    39   ~ 0
-Pi11
-Text Label 3600 3500 2    39   ~ 0
-Pi13
-Text Label 3600 3600 2    39   ~ 0
-Pi15
 Text Label 3600 3800 2    39   ~ 0
 MOSI
@@
 Text Label 4100 3700 0    39   ~ 0
 RT_INIT
-Text Label 4100 3600 0    39   ~ 0
-Pi16
-Text Label 4100 3400 0    39   ~ 0
-Pi12
 Text Label 4100 3300 0    39   ~ 0
 UARTB
@@
 	3300 3300 3300 4100
 Connection ~ 3300 4100
-Text Label 3050 5300 2    39   ~ 0
-Pi7
-Text Label 3050 5500 2    39   ~ 0
-Pi11
-Text Label 3050 5600 2    39   ~ 0
-Pi13
-Text Label 3050 5700 2    39   ~ 0
-Pi15
-Text Label 4950 5700 0    39   ~ 0
-Pi16
 NoConn ~ 1450 1500
 NoConn ~ 1550 1500
@@
 Wire Wire Line
 	5250 4300 5250 4500
-$Comp
-L Connector:TestPoint TP102
-U 1 1 5EA4DCF3
-P 6800 1200
-AR Path="/5EA4DCF3" Ref="TP102"  Part="1"
-AR Path="/5E916134/5EA4DCF3" Ref="TP?"  Part="1"
-AR Path="/5E9D5ED5/5EA4DCF3" Ref="TP?"  Part="1"
-F 0 "TP102" H 6900 1450 50  0000 R CNN
-F 1 "TestPoint" H 6742 1317 50  0001 R CNN
-F 2 "TestPoint:TestPoint_Pad_D1.0mm" H 7000 1200 50  0001 C CNN
-F 3 "~" H 7000 1200 50  0001 C CNN
-	1    6800 1200
-	-1   0    0    1
-$EndComp
-Text Label 6800 1200 2    39   ~ 0
-TGUARD
-$Comp
-L Device:C C101
-U 1 1 5EA4DCFC
-P 6400 1200
-AR Path="/5EA4DCFC" Ref="C101"  Part="1"
-AR Path="/5E916134/5EA4DCFC" Ref="C?"  Part="1"
-F 0 "C101" V 6652 1200 50  0000 C CNN
-F 1 "47uF" V 6561 1200 50  0000 C CNN
-F 2 "Capacitor_SMD:C_0805_2012Metric_Pad1.15x1.40mm_HandSolder" H 6438 1050 50  0001 C CNN
-F 3 "~" H 6400 1200 50  0001 C CNN
-F 4 " C28323" H 6400 1200 50  0001 C CNN "LCSC Part Number"
-F 5 "C0805C105K3RACTU" H 6400 1200 50  0001 C CNN "DigiKey"
-	1    6400 1200
-	0    -1   -1   0
-$EndComp
-$Comp
-L CPU-eagle-import:GND #GND0106
-U 1 1 5EA4DD02
-P 6100 1350
-AR Path="/5EA4DD02" Ref="#GND0106"  Part="1"
-AR Path="/5E916134/5EA4DD02" Ref="#GND?"  Part="1"
-F 0 "#GND0106" H 6100 1350 50  0001 C CNN
-F 1 "GND" H 6100 1340 59  0000 C TNN
-F 2 "" H 6100 1350 50  0001 C CNN
-F 3 "" H 6100 1350 50  0001 C CNN
-	1    6100 1350
-	1    0    0    -1
-$EndComp
-Wire Wire Line
-	6100 1250 6100 1200
-Wire Wire Line
-	6100 1200 6250 1200
-Wire Wire Line
-	6550 1200 6800 1200
 Wire Wire Line
 	4850 1450 4950 1450
@@
 Text Label 4850 1050 0    39   ~ 0
 PI_RESET_TOGGLE
+NoConn ~ 3050 5700
+NoConn ~ 3050 5600
+NoConn ~ 3050 5500
+NoConn ~ 4950 5700
+NoConn ~ 4100 3600
+NoConn ~ 3600 3600
+NoConn ~ 3600 3500
+NoConn ~ 3600 3400
+NoConn ~ 3600 3200
+NoConn ~ 3050 5300
+Text Label 4100 3600 0    39   ~ 0
+Pi16
+Text Label 4100 3400 0    39   ~ 0
+Pi12
+Text Label 3600 3200 2    39   ~ 0
+Pi7
+Text Label 3600 3600 2    39   ~ 0
+Pi15
+Text Label 3600 3500 2    39   ~ 0
+Pi13
+Text Label 3600 3400 2    39   ~ 0
+Pi11
+$Comp
+L power:+3V3 #PWR0102
+U 1 1 5E97A3AA
+P 2950 4950
+F 0 "#PWR0102" H 2950 4800 50  0001 C CNN
+F 1 "+3V3" H 2965 5123 50  0000 C CNN
+F 2 "" H 2950 4950 50  0001 C CNN
+F 3 "" H 2950 4950 50  0001 C CNN
+	1    2950 4950
+	1    0    0    -1
+$EndComp
+Wire Wire Line
+	2950 4950 2950 5800
+NoConn ~ 3050 5000
 $EndSCHEMATC

Commit message: Rewiring the T84 to the 5 volt line.
Changed lines of the file:
@@
 NoConn ~ 1350 1500
 $Sheet
-S 3950 1700 700  350
+S 3950 1700 700  500
 U 5E916134
 F0 "I2C Devices" 39
@@
 F4 "85RES" I L 3950 2000 39
 F5 "SCROLL_INT" I R 4650 1800 39
+F6 "SCL5" I L 3950 2100 39
+F7 "SDA5" I L 3950 2150 39
 $EndSheet
 Text Notes 3200 7250 0    20   ~ 0
@@
 	2950 4950 2950 5800
 NoConn ~ 3050 5000
+Text Label 3950 2100 2    39   ~ 0
+SCL5
+Text Label 3950 2150 2    39   ~ 0
+SDA5
 $EndSCHEMATC

Commit message: Updates from CPU v1 were completed. Switched out Tiny84 for a tiny1614 because the 84 lacks a hardware twi driver. This version was sent to production at jlcpcb.
Parts:
- R101, R102, R103, R104: footprint CPU:R1206 -> Resistor_SMD:R_0805_2012Metric_Pad1.15x1.40mm_HandSolder; DigiKey RC1206FR-0710KL -> RC0805FR-0710KL; LCSC Part Number C17902 -> C17414
Changed lines of the file:
@@
 F 0 "R102" H 7450 2859 59  0000 L BNN
 F 1 "10K" H 7450 2670 59  0000 L BNN
-F 2 "CPU:R1206" H 7600 2800 50  0001 C CNN
+F 2 "Resistor_SMD:R_0805_2012Metric_Pad1.15x1.40mm_HandSolder" H 7600 2800 50  0001 C CNN
 F 3 "" H 7600 2800 50  0001 C CNN
-F 4 " C17902" H 7600 2800 50  0001 C CNN "LCSC Part Number"
-F 5 "RC1206FR-0710KL" H 7600 2800 50  0001 C CNN "DigiKey"
+F 4 " C17414" H 7600 2800 50  0001 C CNN "LCSC Part Number"
+F 5 "RC0805FR-0710KL" H 7600 2800 50  0001 C CNN "DigiKey"
 	1    7600 2800
 	0    -1   -1   0
@@
 F 0 "R104" H 7950 2859 59  0000 L BNN
 F 1 "10K" H 7950 2670 59  0000 L BNN
-F 2 "CPU:R1206" H 8100 2800 50  0001 C CNN
+F 2 "Resistor_SMD:R_0805_2012Metric_Pad1.15x1.40mm_HandSolder" H 8100 2800 50  0001 C CNN
 F 3 "" H 8100 2800 50  0001 C CNN
-F 4 " C17902" H 8100 2800 50  0001 C CNN "LCSC Part Number"
-F 5 "RC1206FR-0710KL" H 8100 2800 50  0001 C CNN "DigiKey"
+F 4 " C17414" H 8100 2800 50  0001 C CNN "LCSC Part Number"
+F 5 "RC0805FR-0710KL" H 8100 2800 50  0001 C CNN "DigiKey"
 	1    8100 2800
 	0    -1   -1   0
@@
 F 0 "R101" H 7450 1709 59  0000 L BNN
 F 1 "10K" H 7450 1520 59  0000 L BNN
-F 2 "CPU:R1206" H 7600 1650 50  0001 C CNN
+F 2 "Resistor_SMD:R_0805_2012Metric_Pad1.15x1.40mm_HandSolder" H 7600 1650 50  0001 C CNN
 F 3 "" H 7600 1650 50  0001 C CNN
-F 4 " C17902" H 7600 1650 50  0001 C CNN "LCSC Part Number"
-F 5 "RC1206FR-0710KL" H 7600 1650 50  0001 C CNN "DigiKey"
+F 4 " C17414" H 7600 1650 50  0001 C CNN "LCSC Part Number"
+F 5 "RC0805FR-0710KL" H 7600 1650 50  0001 C CNN "DigiKey"
 	1    7600 1650
 	0    -1   -1   0
@@
 F 0 "R103" H 7950 1709 59  0000 L BNN
 F 1 "10K" H 7950 1520 59  0000 L BNN
-F 2 "CPU:R1206" H 8100 1650 50  0001 C CNN
+F 2 "Resistor_SMD:R_0805_2012Metric_Pad1.15x1.40mm_HandSolder" H 8100 1650 50  0001 C CNN
 F 3 "" H 8100 1650 50  0001 C CNN
-F 4 " C17902" H 8100 1650 50  0001 C CNN "LCSC Part Number"
-F 5 "RC1206FR-0710KL" H 8100 1650 50  0001 C CNN "DigiKey"
+F 4 " C17414" H 8100 1650 50  0001 C CNN "LCSC Part Number"
+F 5 "RC0805FR-0710KL" H 8100 1650 50  0001 C CNN "DigiKey"
 	1    8100 1650
 	0    -1   -1   0

Commit message: Add display circuitry.
Parts:
- removed J102: Conn_02x14_Odd_Even_MountingPin, CPU:2X14_SMT_MALE-2, symbol Connector_Generic_MountingPin:Conn_02x14_Odd_Even_MountingPin
- added TP102: PiTX, TestPoint:TestPoint_Pad_D1.0mm, symbol Connector:TestPoint
- added TP103: PiRX, TestPoint:TestPoint_Pad_D1.0mm, symbol Connector:TestPoint
- J101: Customer Reference (none) -> CR101-V3; DigiKey NRPN102MAMS-RC,NPPN102FFKS-RC -> NRPN102MAMS-RC
- Pi101: Customer Reference (none) -> CR101-V3; DigiKey (none) -> 609-2231-ND
- Q101, Q102, R101, R102, R103, R104, SW101, TP101: Customer Reference (none) -> CR101-V3
Connections:
- net labels added: LCD_BACK_LIGHT, PiRX, PiTX
- net labels removed: Pi11, Pi12, Pi13, Pi15, Pi16, Pi7, UARTA, UARTB
- wire segments 102 -> 86
- no-connect marks 29 -> 19
Changed lines of the file:
@@
 $Descr User 11693 8394
 encoding utf-8
-Sheet 1 3
+Sheet 1 4
 Title ""
 Date ""
@@
 F 2 "CPU:RASPBERRYPI_Zero-No_Mounting_Holes_SMD_Flat" H 3950 6200 50  0001 C CNN
 F 3 "" H 3950 6200 50  0001 C CNN
+F 4 "609-2231-ND" H 3950 6200 50  0001 C CNN "DigiKey"
+F 5 "CR101-V3" H 3950 6200 50  0001 C CNN "Customer Reference"
 	1    3950 6200
 	1    0    0    -1
@@
 F 3 "~" H 1850 1700 50  0001 C CNN
 F 4 "C135211" H 1850 1700 50  0001 C CNN "LCSC Part Number"
-F 5 "NRPN102MAMS-RC,NPPN102FFKS-RC" H 1850 1700 50  0001 C CNN "DigiKey"
+F 5 "NRPN102MAMS-RC" H 1850 1700 50  0001 C CNN "DigiKey"
+F 6 "CR101-V3" H 1850 1700 50  0001 C CNN "Customer Reference"
 	1    1850 1700
 	0    1    1    0
 $EndComp
 Text Label 4950 5300 0    39   ~ 0
-UARTA
+PiTX
 Text Label 4950 5400 0    39   ~ 0
-UARTB
+PiRX
 Wire Wire Line
 	1650 1500 1650 1400
@@
 Text Label 4950 5800 0    39   ~ 0
 RT_INIT
-$Comp
-L Connector_Generic_MountingPin:Conn_02x14_Odd_Even_MountingPin J102
-U 1 1 5EA0CFAA
-P 3800 3500
-F 0 "J102" H 3850 4317 50  0000 C CNN
-F 1 "Conn_02x14_Odd_Even_MountingPin" H 3850 4226 50  0000 C CNN
-F 2 "CPU:2X14_SMT_MALE-2" H 3800 3500 50  0001 C CNN
-F 3 "~" H 3800 3500 50  0001 C CNN
-	1    3800 3500
-	1    0    0    -1
-$EndComp
-$Comp
-L power:+3V3 #PWR0103
-U 1 1 5EB169CB
-P 3500 2700
-F 0 "#PWR0103" H 3500 2550 50  0001 C CNN
-F 1 "+3V3" H 3515 2873 50  0000 C CNN
-F 2 "" H 3500 2700 50  0001 C CNN
-F 3 "" H 3500 2700 50  0001 C CNN
-	1    3500 2700
-	1    0    0    -1
-$EndComp
-Wire Wire Line
-	3400 3700 3400 2900
-Wire Wire Line
-	3600 2900 3500 2900
-Wire Wire Line
-	3500 2900 3500 2700
-Wire Wire Line
-	3400 3700 3600 3700
-Wire Wire Line
-	3500 2900 3400 2900
-Connection ~ 3500 2900
-Text Label 3600 3800 2    39   ~ 0
-MOSI
-Text Label 3600 3900 2    39   ~ 0
-MISO
-Text Label 3600 4000 2    39   ~ 0
-SCLK
-Text Label 3600 4200 2    39   ~ 0
-EEDATA
-Text Label 4100 4200 0    39   ~ 0
-EECLK
-Text Label 4100 4100 0    39   ~ 0
-RT_CS
-Text Label 4100 4000 0    39   ~ 0
-TFT_CS
-Text Label 4100 3900 0    39   ~ 0
-TFT_DC
-Text Label 4100 3700 0    39   ~ 0
-RT_INIT
-Text Label 4100 3300 0    39   ~ 0
-UARTB
-Text Label 4100 3200 0    39   ~ 0
-UARTA
-Text Label 4100 3000 0    39   ~ 0
-Pi5V
-Text Label 4100 2900 0    39   ~ 0
-Pi5V
-Wire Wire Line
-	4100 2900 4200 2900
-Wire Wire Line
-	4100 3000 4200 3000
-Wire Wire Line
-	4200 3000 4200 2900
-$Comp
-L CPU-eagle-import:GND #GND0104
-U 1 1 5EB810B6
-P 4400 4000
-F 0 "#GND0104" H 4400 4000 50  0001 C CNN
-F 1 "GND" H 4400 4000 59  0000 C TNN
-F 2 "" H 4400 4000 50  0001 C CNN
-F 3 "" H 4400 4000 50  0001 C CNN
-	1    4400 4000
-	1    0    0    -1
-$EndComp
-Wire Wire Line
-	4100 3100 4400 3100
-Wire Wire Line
-	4400 3100 4400 3500
-Wire Wire Line
-	4100 3800 4400 3800
-Connection ~ 4400 3800
-Wire Wire Line
-	4400 3800 4400 3900
-Wire Wire Line
-	4100 3500 4400 3500
-Connection ~ 4400 3500
-Wire Wire Line
-	4400 3500 4400 3800
-$Comp
-L CPU-eagle-import:GND #GND0103
-U 1 1 5EBAA119
-P 3300 4200
-F 0 "#GND0103" H 3300 4200 50  0001 C CNN
-F 1 "GND" H 3300 4200 59  0000 C TNN
-F 2 "" H 3300 4200 50  0001 C CNN
-F 3 "" H 3300 4200 50  0001 C CNN
-	1    3300 4200
-	1    0    0    -1
-$EndComp
-Wire Wire Line
-	3600 4100 3300 4100
-Wire Wire Line
-	3600 3300 3300 3300
-Wire Wire Line
-	3300 3300 3300 4100
-Connection ~ 3300 4100
 NoConn ~ 1450 1500
 NoConn ~ 1550 1500
@@
 F 4 "C221841" H 5150 4700 50  0001 C CNN "LCSC Part Number"
 F 5 "PCM12SMTR" H 5150 4700 50  0001 C CNN "DigiKey"
+F 6 "CR101-V3" H 5150 4700 50  0001 C CNN "Customer Reference"
 	1    5150 4700
 	0    -1   -1   0
@@
 Text Label 5150 5000 0    39   ~ 0
 Pi5V
-NoConn ~ 3850 4400
 NoConn ~ 5050 4500
 NoConn ~ 3050 6400
@@
 F 4 "C67273" H 7850 3100 50  0001 C CNN "LCSC Part Number"
 F 5 "IRLML0040TRPBF" H 7850 3100 50  0001 C CNN "DigiKey"
+F 6 "CR101-V3" H 7850 3100 50  0001 C CNN "Customer Reference"
 	1    7850 3100
 	0    1    1    0
@@
 F 4 " C17414" H 7600 2800 50  0001 C CNN "LCSC Part Number"
 F 5 "RC0805FR-0710KL" H 7600 2800 50  0001 C CNN "DigiKey"
+F 6 "CR101-V3" H 7600 2800 50  0001 C CNN "Customer Reference"
 	1    7600 2800
 	0    -1   -1   0
@@
 F 4 " C17414" H 8100 2800 50  0001 C CNN "LCSC Part Number"
 F 5 "RC0805FR-0710KL" H 8100 2800 50  0001 C CNN "DigiKey"
+F 6 "CR101-V3" H 8100 2800 50  0001 C CNN "Customer Reference"
 	1    8100 2800
 	0    -1   -1   0
@@
 F 4 "C67273" H 7850 1950 50  0001 C CNN "LCSC Part Number"
 F 5 "IRLML0040TRPBF" H 7850 1950 50  0001 C CNN "DigiKey"
+F 6 "CR101-V3" H 7850 1950 50  0001 C CNN "Customer Reference"
 	1    7850 1950
 	0    1    1    0
@@
 F 4 " C17414" H 7600 1650 50  0001 C CNN "LCSC Part Number"
 F 5 "RC0805FR-0710KL" H 7600 1650 50  0001 C CNN "DigiKey"
+F 6 "CR101-V3" H 7600 1650 50  0001 C CNN "Customer Reference"
 	1    7600 1650
 	0    -1   -1   0
@@
 F 4 " C17414" H 8100 1650 50  0001 C CNN "LCSC Part Number"
 F 5 "RC0805FR-0710KL" H 8100 1650 50  0001 C CNN "DigiKey"
+F 6 "CR101-V3" H 8100 1650 50  0001 C CNN "Customer Reference"
 	1    8100 1650
 	0    -1   -1   0
@@
 Wire Wire Line
 	2550 6900 2450 6900
-$Comp
-L power:PWR_FLAG #FLG0103
-U 1 1 5EB569E1
-P 3300 2900
-F 0 "#FLG0103" H 3300 2975 50  0001 C CNN
-F 1 "PWR_FLAG" V 3300 3027 50  0000 L CNN
-F 2 "" H 3300 2900 50  0001 C CNN
-F 3 "~" H 3300 2900 50  0001 C CNN
-	1    3300 2900
-	0    -1   -1   0
-$EndComp
-Wire Wire Line
-	3400 2900 3300 2900
-Connection ~ 3400 2900
 Wire Wire Line
 	1450 2000 1450 2400
@@
 Text Notes 3200 7250 0    20   ~ 0
 I2C slave setup:\nhttps://raspberrypi.stackexchange.com/questions/76109/raspberry-as-an-i2c-slave
-NoConn ~ 4100 3400
-NoConn ~ 3600 3100
-NoConn ~ 3600 3000
 NoConn ~ 3050 5100
 NoConn ~ 3050 5200
@@
 F 2 "TestPoint:TestPoint_Pad_D1.0mm" H 5150 3300 50  0001 C CNN
 F 3 "~" H 5150 3300 50  0001 C CNN
+F 4 "CR101-V3" H 4950 3300 50  0001 C CNN "Customer Reference"
 	1    4950 3300
 	1    0    0    -1
@@
 NoConn ~ 3050 5600
 NoConn ~ 3050 5500
-NoConn ~ 4950 5700
-NoConn ~ 4100 3600
-NoConn ~ 3600 3600
-NoConn ~ 3600 3500
-NoConn ~ 3600 3400
-NoConn ~ 3600 3200
 NoConn ~ 3050 5300
-Text Label 4100 3600 0    39   ~ 0
-Pi16
-Text Label 4100 3400 0    39   ~ 0
-Pi12
-Text Label 3600 3200 2    39   ~ 0
-Pi7
-Text Label 3600 3600 2    39   ~ 0
-Pi15
-Text Label 3600 3500 2    39   ~ 0
-Pi13
-Text Label 3600 3400 2    39   ~ 0
-Pi11
 $Comp
 L power:+3V3 #PWR0102
@@
 Text Label 3950 2150 2    39   ~ 0
 SDA5
+$Sheet
+S 5550 1800 850  1050
+U 5EC4945A
+F0 "Display" 39
+F1 "Display.sch" 39
+F2 "MOSI" I L 5550 1900 39
+F3 "MISO" I L 5550 2000 39
+F4 "SCLK" I L 5550 2100 39
+F5 "EEDATA" I L 5550 2200 39
+F6 "EECLK" I L 5550 2300 39
+F7 "RT_CS" I L 5550 2400 39
+F8 "TFT_CS" I L 5550 2500 39
+F9 "TFT_DC" I L 5550 2600 39
+F10 "RT_INIT" I L 5550 2700 39
+F11 "GPIO23" I L 5550 2800 39
+F12 "Pi5V" I R 6400 2300 39
+$EndSheet
+Text Label 5550 2700 2    39   ~ 0
+RT_INIT
+Text Label 5550 2600 2    39   ~ 0
+TFT_DC
+Text Label 5550 2500 2    39   ~ 0
+TFT_CS
+Text Label 5550 2400 2    39   ~ 0
+RT_CS
+Text Label 5550 2300 2    39   ~ 0
+EECLK
+Text Label 5550 2200 2    39   ~ 0
+EEDATA
+Text Label 5550 2100 2    39   ~ 0
+SCLK
+Text Label 5550 2000 2    39   ~ 0
+MISO
+Text Label 5550 1900 2    39   ~ 0
+MOSI
+Text Label 5550 2800 2    39   ~ 0
+LCD_BACK_LIGHT
+Text Label 4950 5700 0    39   ~ 0
+LCD_BACK_LIGHT
+$Comp
+L Connector:TestPoint TP102
+U 1 1 5EE03ABB
+P 5550 5300
+F 0 "TP102" H 5500 5550 50  0000 L CNN
+F 1 "PiTX" V 5500 5250 50  0000 L CNN
+F 2 "TestPoint:TestPoint_Pad_D1.0mm" H 5750 5300 50  0001 C CNN
+F 3 "~" H 5750 5300 50  0001 C CNN
+F 4 "CR101-V3" H 5550 5300 50  0001 C CNN "Customer Reference"
+	1    5550 5300
+	0    1    1    0
+$EndComp
+Wire Wire Line
+	4950 5300 5550 5300
+$Comp
+L Connector:TestPoint TP103
+U 1 1 5EE07231
+P 5550 5400
+F 0 "TP103" H 5500 5650 50  0000 L CNN
+F 1 "PiRX" V 5600 5400 50  0000 L CNN
+F 2 "TestPoint:TestPoint_Pad_D1.0mm" H 5750 5400 50  0001 C CNN
+F 3 "~" H 5750 5400 50  0001 C CNN
+F 4 "CR101-V3" H 5550 5400 50  0001 C CNN "Customer Reference"
+	1    5550 5400
+	0    1    1    0
+$EndComp
+Wire Wire Line
+	4950 5400 5550 5400
+Text Label 6400 2300 0    39   ~ 0
+Pi5V
 $EndSCHEMATC
